Commit message: Urdf with mass

File: robots/monoped_description/urdf/monoped.urdf (robot description, URDF)
Before this commit: robot monoped, 4 links, 3 joints
Links:
- added link lowerleg_contactsensor_link, mass 0.01; collision sphere radius=0.020; visual sphere radius=0.020
- link base: mass None -> 0.18; geometry collision box size=0.20 0.20 0.30; visual box size=0.20 0.20 0.30
- link hipassembly: mass None -> 0.18; geometry collision mesh filename=package://example-robot-data/robots/monoped_description/hip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 scale=1 1 1; visual mesh filename=package://example-robot-data/robots/monoped_description/hip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 scale=1 1 1
- link lowerleg: mass None -> 0.18; geometry collision mesh filename=package://example-robot-data/robots/monoped_description/low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 scale=1 1 1; visual mesh filename=package://example-robot-data/robots/monoped_description/low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 scale=1 1 1
- link upperleg: mass None -> 0.18; geometry collision mesh filename=package://example-robot-data/robots/monoped_description/upp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 scale=1 1 1; visual mesh filename=package://example-robot-data/robots/monoped_description/upp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 scale=1 1 1
Joints:
- added joint lowerleg_contactsensor_link_joint: type fixed, parent lowerleg, child lowerleg_contactsensor_link, origin xyz=0.35 0 0 rpy=0 0 0
- joint haa_joint: limit lower=-1.6 upper=1.6 effort=200 velocity=1.0 -> lower=-1.6 upper=1.6 effort=200 velocity=10.0
- joint hfe_joint: limit lower=-1.6 upper=1.6 effort=200 velocity=1.0 -> lower=-1.6 upper=1.6 effort=200 velocity=10.0
- joint kfe_joint: limit lower=-1.6 upper=1.6 effort=200 velocity=1.0 -> lower=-1.6 upper=1.6 effort=200 velocity=10.0

Commit message: CHange foot name + reference state

File: robots/monoped_description/urdf/monoped.urdf (robot description, URDF)
Before this commit: robot monoped, 5 links, 4 joints
Links:
- removed link lowerleg_contactsensor_link
- added link foot_link, mass 0.01; collision sphere radius=0.020; visual sphere radius=0.020
- link hipassembly: geometry collision mesh filename=package://example-robot-data/robots/monoped_description/vis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 scale=1 1 1; visual mesh filename=package://example-robot-data/robots/monoped_description/vis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 scale=1 1 1
- link lowerleg: geometry collision mesh filename=package://example-robot-data/robots/monoped_description/vis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 scale=1 1 1; visual mesh filename=package://example-robot-data/robots/monoped_description/vis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 scale=1 1 1
- link upperleg: geometry collision mesh filename=package://example-robot-data/robots/monoped_description/vis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 scale=1 1 1; visual mesh filename=package://example-robot-data/robots/monoped_description/vis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 scale=1 1 1
Joints:
- removed joint lowerleg_contactsensor_link_joint
- added joint foot_link_joint: type fixed, parent lowerleg, child foot_link, origin xyz=0.35 0 0 rpy=0 0 0
